File: current-monitor.kicad_pcb (KiCad board)
At the start: 4 copper layers, 100 x 70 mm, 152 parts, among them J201 CONN-3, J601 USB-MICROB, J602 JTAG, J603 CONN-6, K201 RELAY-DPDT-EE2-SPLIT, K202 RELAY-DPDT-EE2-SPLIT, Q201 DRDC3105E6, U201 FSA1259A, U202 MAX4737EUD, U301 AD8429A, U302 TL032C, U303 LM833, U401 INA826, U501 TL032C, U601 K22F-64LQFP, U701 LM27313, U702 MAX6070, U703 LTC3260MSE, Y601 4MHz

Commit message: checkpoint
Connections:
- S601 pad 1: (no net) -> COM
- S601 pad 2: COM -> (no net)
- S601 pad 3: (no net) -> /MCU/~RESET
- S601 pad 4: /MCU/~RESET -> (no net)
Routing:
- net +5V: track 147.3 -> 54.1 mm, vias 8 -> 12
- net -Vs: track 103.3 -> 68.6 mm, vias 10 -> 11
- net /Current Sense Coarse Range/SENSE_COARSE: track 15.1 -> 20.6 mm
- net /MCU/SENSE_VOLTAGE: track 16.5 -> 21.9 mm
- net /MCU/~RESET: track 21.7 -> 26.1 mm, vias 2 -> 3
- net SENSE+: track 85.4 -> 89.2 mm
- net /Power Supply/-Vs_UNREG: track 3.61 -> 6.83 mm
- net /Current Sense Fine Range/SENSE_FINE: track 11.9 -> 15.1 mm
- net +3.00V: track 88.2 -> 91.0 mm, vias 1 -> 2
- net SENSE-: track 61.4 -> 64.2 mm
- net /Sense Voltage/VOLTAGE_RAW: track 39.0 -> 41.1 mm
- net /MCU/5V_MCU: track 33.2 -> 34.9 mm
- net /Power Supply/+Vs_UNREG: track 16.4 -> 17.8 mm
- net /Current Sense Coarse Range/COARSE_UNCLAMPED: track 21.3 -> 22.4 mm
- net /Current Sense Fine Range/REF_ADJUST: track 23.1 -> 24.2 mm
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- added copper zone on In2.Cu, net +3V3
- added copper zone on In2.Cu, net +5V
- added copper zone on In2.Cu, net +Vs
- added copper zone on In2.Cu, net -Vs

Commit message: full design
Parts:
- J602: value JTAG -> SWD
- moved TP401 11.2 mm to (109.6, 113.6)
Other:
- board size 100 x 70 mm -> 70 x 58.2 mm
