File: current-monitor.kicad_pcb (KiCad board)
At the start: 4 copper layers, 70 x 58.2 mm, 152 parts, among them J201 CONN-3, J601 USB-MICROB, J602 SWD, J603 CONN-6, K201 RELAY-DPDT-EE2-SPLIT, K202 RELAY-DPDT-EE2-SPLIT, Q201 DRDC3105E6, U201 FSA1259A, U202 MAX4737EUD, U301 AD8429A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

Commit message: case size pass
Parts:
- moved C610 0.80 mm to (156.2, 83.6)
- moved R603 0.80 mm to (156.2, 82.0)
Changed lines of the file:
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@@
     (thickness 1.6)
     (drawings 14)
-    (tracks 1231)
+    (tracks 1233)
     (zones 0)
     (modules 152)
@@
     (46 B.CrtYd user)
     (47 F.CrtYd user)
-    (49 F.Fab user)
+    (49 F.Fab user hide)
   )
   (setup
-    (last_trace_width 0.2)
+    (last_trace_width 0.25)
     (user_trace_width 0.2)
     (user_trace_width 0.25)
@@
   )
   (module libs:SMD-1608 (layer F.Cu)
-    (at 156.2 82.8 270)
+    (at 156.2 82 270)
     (fp_text reference R603 (at -2.2 1.4 360) (layer F.SilkS)
       (effects (font (size 0.7 0.7) (thickness 0.15)))
@@
   )
   (module libs:SMD-1608 (layer F.Cu)
-    (at 156.2 84.4 90)
+    (at 156.2 83.6 90)
     (fp_text reference C610 (at 2.8 -1.4 180) (layer F.SilkS)
       (effects (font (size 0.7 0.7) (thickness 0.15)))
@@
   (segment (start 103.705 91.055) (end 103.65 91) (width 0.4) (layer F.Cu) (net 1))
   (segment (start 103.65 91) (end 102.8 91) (width 0.4) (layer F.Cu) (net 1) (status 20))
+  (via (at 157.8 83.599998) (size 0.6) (drill 0.3) (layers F.Cu B.Cu) (net 2))
   (segment (start 154.45 73.15) (end 153.8 73.8) (width 0.5) (layer F.Cu) (net 2) (status 10))
   (segment (start 154.55 73.15) (end 154.45 73.15) (width 0.5) (layer F.Cu) (net 2) (status 30))
@@
   (segment (start 153.360881 112.760881) (end 153.4 112.8) (width 0.5) (layer F.Cu) (net 2))
   (via (at 153.4 112.8) (size 0.6) (drill 0.3) (layers F.Cu B.Cu) (net 2))
-  (segment (start 157 84.4) (end 157.8 84.4) (width 0.25) (layer F.Cu) (net 2) (status 10))
-  (via (at 157.8 84.4) (size 0.6) (drill 0.3) (layers F.Cu B.Cu) (net 2))
+  (segment (start 157 83.6) (end 157.8 83.6) (width 0.25) (layer F.Cu) (net 2) (status 10))
   (segment (start 155.8 96) (end 155.8 95.4) (width 0.4) (layer F.Cu) (net 2))
   (via (at 155.8 95.4) (size 0.6) (drill 0.3) (layers F.Cu B.Cu) (net 2))
@@
   (segment (start 132.55 95.25) (end 132.55 93.85) (width 0.5) (layer F.Cu) (net 12) (status 30))
   (segment (start 132.55 93.85) (end 132.6 93.8) (width 0.5) (layer F.Cu) (net 12) (status 30))
+  (segment (start 148.8 89.291478) (end 156.091496 81.999982) (width 0.5) (layer In2.Cu) (net 13))
+  (segment (start 148.8 90) (end 148.8 89.291478) (width 0.5) (layer In2.Cu) (net 13))
+  (segment (start 157.375736 81.999982) (end 157.8 81.999982) (width 0.5) (layer In2.Cu) (net 13))
+  (segment (start 156.091496 81.999982) (end 157.375736 81.999982) (width 0.5) (layer In2.Cu) (net 13))
+  (via (at 157.8 81.999982) (size 0.6) (drill 0.3) (layers F.Cu B.Cu) (net 13))
   (segment (start 135.2 88.8) (end 136 88) (width 0.5) (layer In2.Cu) (net 13))
   (segment (start 136 88) (end 136 78.6) (width 0.5) (layer In2.Cu) (net 13))
@@
   (segment (start 128.6 83.308522) (end 133.308522 78.6) (width 0.5) (layer In2.Cu) (net 13))
   (segment (start 133.308522 78.6) (end 136 78.6) (width 0.5) (layer In2.Cu) (net 13))
-  (segment (start 148.8 90) (end 148.8 89.291478) (width 0.5) (layer In2.Cu) (net 13))
-  (segment (start 148.8 89.291478) (end 155.291478 82.8) (width 0.5) (layer In2.Cu) (net 13))
-  (segment (start 155.291478 82.8) (end 157.8 82.8) (width 0.5) (layer In2.Cu) (net 13))
   (segment (start 143.161154 78.6) (end 145.491478 78.6) (width 0.5) (layer In2.Cu) (net 13))
   (segment (start 138.4 78.6) (end 143.161154 78.6) (width 0.5) (layer In2.Cu) (net 13))
@@
   (segment (start 138.4 77.8) (end 138.4 78.6) (width 0.5) (layer F.Cu) (net 13) (status 10))
   (via (at 138.4 78.6) (size 0.6) (drill 0.3) (layers F.Cu B.Cu) (net 13))
-  (segment (start 157 82.8) (end 157.8 82.8) (width 0.25) (layer F.Cu) (net 13) (status 10))
-  (via (at 157.8 82.8) (size 0.6) (drill 0.3) (layers F.Cu B.Cu) (net 13))
+  (segment (start 157 82) (end 157.8 82) (width 0.25) (layer F.Cu) (net 13) (status 10))
   (segment (start 153.4 77.8) (end 154.2 77.8) (width 0.5) (layer F.Cu) (net 13) (status 10))
   (via (at 154.2 77.8) (size 0.6) (drill 0.3) (layers F.Cu B.Cu) (net 13))
@@
   (segment (start 148.65 87.35) (end 148.65 89.05) (width 0.3) (layer F.Cu) (net 13) (status 30))
   (segment (start 148.65 89.05) (end 148.8 89.2) (width 0.3) (layer F.Cu) (net 13) (status 30))
+  (segment (start 151.6 84.9) (end 152.6 84.9) (width 0.25) (layer F.Cu) (net 14))
+  (segment (start 152.6 84.9) (end 153.9 83.6) (width 0.25) (layer F.Cu) (net 14))
+  (segment (start 153.9 83.6) (end 155.4 83.6) (width 0.25) (layer F.Cu) (net 14))
   (segment (start 143.2 97.6) (end 142.6 97.6) (width 0.2) (layer F.Cu) (net 14) (status 20))
   (segment (start 142.6 97.6) (end 142.5 97.5) (width 0.2) (layer F.Cu) (net 14) (status 30))
@@
   (segment (start 150.494328 84.9) (end 150.494294 84.900034) (width 0.25) (layer F.Cu) (net 14))
   (via (at 150.494294 84.900034) (size 0.6) (drill 0.3) (layers F.Cu B.Cu) (net 14))
-  (segment (start 151.6 84.9) (end 154.9 84.9) (width 0.25) (layer F.Cu) (net 14) (status 10))
-  (segment (start 154.9 84.9) (end 155.4 84.4) (width 0.25) (layer F.Cu) (net 14) (status 20))
-  (segment (start 155.4 82.8) (end 155.4 84.4) (width 0.25) (layer F.Cu) (net 14) (status 30))
+  (segment (start 155.4 82) (end 155.4 83.6) (width 0.25) (layer F.Cu) (net 14) (status 30))
   (segment (start 154.6 79.834996) (end 154.6 96.8) (width 0.25) (layer B.Cu) (net 15))
   (segment (start 154.846951 97.046951) (end 154.857426 97.046951) (width 0.25) (layer B.Cu) (net 15))
@@
     (connect_pads yes (clearance 0.2))
     (min_thickness 0.254)
-    (fill yes (arc_segments 32) (thermal_gap 0.508) (thermal_bridge_width 0.508))
+    (fill (arc_segments 32) (thermal_gap 0.508) (thermal_bridge_width 0.508))
     (polygon
       (pts
@@
     (connect_pads yes (clearance 0.2))
     (min_thickness 0.254)
-    (fill yes (arc_segments 32) (thermal_gap 0.508) (thermal_bridge_width 0.508))
+    (fill (arc_segments 32) (thermal_gap 0.508) (thermal_bridge_width 0.508))
     (polygon
       (pts
@@
     (connect_pads yes (clearance 0.2))
     (min_thickness 0.254)
-    (fill yes (arc_segments 32) (thermal_gap 0.508) (thermal_bridge_width 0.508))
+    (fill (arc_segments 32) (thermal_gap 0.508) (thermal_bridge_width 0.508))
     (polygon
       (pts
@@
     (connect_pads yes (clearance 0.2))
     (min_thickness 0.254)
-    (fill yes (arc_segments 32) (thermal_gap 0.508) (thermal_bridge_width 0.508))
+    (fill (arc_segments 32) (thermal_gap 0.508) (thermal_bridge_width 0.508))
     (polygon
       (pts
@@
     (connect_pads yes (clearance 0.2))
     (min_thickness 0.254)
-    (fill yes (arc_segments 32) (thermal_gap 0.508) (thermal_bridge_width 0.508))
+    (fill (arc_segments 32) (thermal_gap 0.508) (thermal_bridge_width 0.508))
     (polygon
       (pts
@@
     (connect_pads yes (clearance 0.2))
     (min_thickness 0.254)
-    (fill yes (arc_segments 32) (thermal_gap 0.508) (thermal_bridge_width 0.508))
+    (fill (arc_segments 32) (thermal_gap 0.508) (thermal_bridge_width 0.508))
     (polygon
       (pts
@@
     (connect_pads yes (clearance 0.2))
     (min_thickness 0.254)
-    (fill yes (arc_segments 32) (thermal_gap 0.2) (thermal_bridge_width 0.508))
+    (fill (arc_segments 32) (thermal_gap 0.2) (thermal_bridge_width 0.508))
     (polygon
       (pts
@@
     (connect_pads yes (clearance 0.2))
     (min_thickness 0.254)
-    (fill yes (arc_segments 32) (thermal_gap 0.508) (thermal_bridge_width 0.508))
+    (fill (arc_segments 32) (thermal_gap 0.508) (thermal_bridge_width 0.508))
     (polygon
       (pts
@@
     (connect_pads yes (clearance 0.2))
     (min_thickness 0.254)
-    (fill yes (arc_segments 32) (thermal_gap 0.508) (thermal_bridge_width 0.508))
+    (fill (arc_segments 32) (thermal_gap 0.508) (thermal_bridge_width 0.508))
     (polygon
       (pts
@@
     (connect_pads yes (clearance 0.2))
     (min_thickness 0.254)
-    (fill yes (arc_segments 32) (thermal_gap 0.508) (thermal_bridge_width 0.508))
+    (fill (arc_segments 32) (thermal_gap 0.508) (thermal_bridge_width 0.508))
     (polygon
       (pts
@@
     (connect_pads yes (clearance 0.2))
     (min_thickness 0.254)
-    (fill yes (arc_segments 32) (thermal_gap 0.508) (thermal_bridge_width 0.508))
+    (fill (arc_segments 32) (thermal_gap 0.508) (thermal_bridge_width 0.508))
     (polygon
       (pts
@@
     (connect_pads yes (clearance 0.2))
     (min_thickness 0.254)
-    (fill yes (arc_segments 32) (thermal_gap 0.508) (thermal_bridge_width 0.508))
+    (fill (arc_segments 32) (thermal_gap 0.508) (thermal_bridge_width 0.508))
     (polygon
       (pts
@@
     (connect_pads yes (clearance 0.2))
     (min_thickness 0.254)
-    (fill yes (arc_segments 32) (thermal_gap 0.508) (thermal_bridge_width 0.508))
+    (fill (arc_segments 32) (thermal_gap 0.508) (thermal_bridge_width 0.508))
     (polygon
       (pts
@@
     (connect_pads yes (clearance 0.2))
     (min_thickness 0.254)
-    (fill yes (arc_segments 32) (thermal_gap 0.508) (thermal_bridge_width 0.508))
+    (fill (arc_segments 32) (thermal_gap 0.508) (thermal_bridge_width 0.508))
     (polygon
       (pts

Commit message: adapt layout
Parts:
- C201, C708: footprint libs:SMD-2012 -> libs:SMD-3225
- C205, C207: value 10n -> 4.7n
- C206: value 100n -> 47n
- C306, C308, C404: value C -> 1n; footprint libs:SMD-2012 -> libs:SMD-1608
- C307: value 0.47n -> 470p
- C311, C407, C703, C710, C711: footprint libs:SMD-2012 -> libs:SMD-1608
- C312, C408: value C -> 4.7n
- C403: value C -> 120p; footprint libs:SMD-2012 -> libs:SMD-1608
- C503: value 4n -> 4.7n
- C601, C602: value C -> 8p
- C603, C709: value 1u -> 2.2u
- C704: value 115p -> 120p
- C706, C707, C712, C713: value 4.7u -> 10u; footprint libs:SMD-2012 -> libs:SMD-3225
- F201: value FUSE -> 2A
- L601, L702: value LCORE -> MPZ1608B471ATA00
- L701: value 22u -> 33u 0.2A
- R209, R210: value 33 -> 10
- R305: value Rs -> 4.9k
- R306: value Rs -> 2.36k
- R309: value R -> 4.7k
- R310: value R -> 9.4k
- R313, R406: value R -> 971
- R402: value Rs -> 6.66k
- R403: value Rs -> 14.5k
- R405: value 470 -> 499
- Y601: value 4MHz -> 10MHz
- moved R207 2.84 mm to (118.2, 76.6)
- moved C201 2.42 mm to (115.6, 76.6)
- moved C707 1.73 mm to (146.8, 105.2)
- moved C708 1.63 mm to (146.7, 112.2)
- moved C706 0.94 mm to (151.8, 112.4)
- moved C712 0.60 mm to (142.6, 102.6)
- moved TP703 0.60 mm to (145.8, 115.4)
- moved C713 0.52 mm to (142.6, 114.5)
- turned SJ702 to 180 degrees
- turned SJ703 to 180 degrees
- renumbered R704 to SJ702, R705 to SJ703
Connections:
- SJ702 pad 1: /Power Supply/+Vs_UNREG -> Net-(SJ702-Pad1)
- SJ702 pad 2: Net-(R704-Pad2) -> /Power Supply/+Vs_UNREG
- SJ703 pad 1: Net-(R704-Pad2) -> COM
- SJ703 pad 2: COM -> Net-(SJ702-Pad1)
- U703 pad 14: Net-(R704-Pad2) -> Net-(SJ702-Pad1)
Routing:
- net Net-(R704-Pad2): track 8.91 -> 0.00 mm, vias 3 -> 0
- net Net-(SJ702-Pad1): track 0.00 -> 8.90 mm, vias 0 -> 2
- net +Vs: track 85.3 -> 83.8 mm, vias 11 -> 9
- net /Power Supply/+Vs_UNREG: track 17.8 -> 19.1 mm
- net /In/Out, Shunt, Calibration/IN: track 59.2 -> 57.9 mm
- net /Power Supply/-Vs_UNREG: track 6.83 -> 7.90 mm
- net COM: track 114.8 -> 114.4 mm, vias 110 -> 107
- net -Vs: track 68.6 -> 68.9 mm, vias 11 -> 9
